File: prod/BasilBoxHardware/led_light_control.kicad_sch (KiCad schematic)
At the start: 2 parts, among them U4 DEBO_Mosfet, U5 LED_LIGHT

Commit message: Add hardware schematics
Connections:
- new net: U4. (TRIG), U5. (DIM-)
